File: fileOperation.sch (KiCad schematic (older format))
At the start: 13 parts, among them IC1 XC95288XL-10TQ144I, J1 Conn_01x05_Male, J4 Conn_02x21_Odd_Even

Commit message: Replacing CPLD, add 1.8V regulator, see CHANGELOG
Parts:
- removed IC1: XC95288XL-10TQ144I, Package_QFP:TQFP-144_20x20mm_P0.5mm, symbol XC95288XL-10TQ144I:XC95288XL-10TQ144I
- removed J1: Conn_01x05_Male, Connector_PinHeader_2.54mm:PinHeader_1x05_P2.54mm_Vertical, symbol Connector:Conn_01x05_Male
- removed J4: Conn_02x21_Odd_Even, Connector_PinHeader_1.27mm:PinHeader_2x21_P1.27mm_Vertical, symbol Connector_Generic:Conn_02x21_Odd_Even
- added IC1: XC2C256-VQ100, symbol FPGA_Xilinx:XC2C256-VQ100
- added J1: ALU_JTAG, symbol Connector:Conn_01x06_Male
- added J4: UnusedPins_Connector, symbol Connector_Generic:Conn_02x15_Odd_Even
- added J5: ALU_PINS, symbol Connector_Generic:Conn_02x19_Odd_Even
- added U28: TPS7A0518PDBZR, symbol Custom:TPS7A0518PDBZR
- C20, C24, C26, C28, C32, C39, C7, C9: value 10nF -> 100nF
- C33, C40: value 10nF -> 1uF
Connections:
- net labels added: +1V8
- net labels removed: UNUSED_D4, UNUSED_D5, UNUSED_D6, UNUSED_D7, UNUSED_E0, UNUSED_E1, UNUSED_E2, UNUSED_E3, UNUSED_E4, UNUSED_E5, UNUSED_E6, UNUSED_E7
- wire segments 217 -> 135
- no-connect marks 42 -> 17
Other:
- moved on the sheet: C20, C24, C26, C28, C32, C39, C7, C9

Commit message: Adding SN74LVC8T245DW and SN74AVC4T245D
Parts:
- added C44, C45: 10nF, Capacitor_SMD:C_0805_2012Metric, symbol Device:C
- added U30: SN74LVC8T245DW, symbol Custom:SN74LVC8T245DW
- added U32: SN74AVC4T245D, symbol Custom:SN74AVC4T245D
Connections:
- net +3V3: now also C44.2, C45.2, U30.1 (VCCA), U30.2 (DIR), U30.23 (VCCB), U30.24 (VCCB), U32.1 (VCCA), U32.16 (VCCB), U32.2 (1DIR), U32.3 (2DIR)
- net DLEFT_0: now also U30.21 (B1)
- net DLEFT_1: now also U30.20 (B2)
- net DLEFT_2: now also U30.19 (B3)
- net DLEFT_3: now also U30.18 (B4)
- net DLEFT_4: now also U30.17 (B5)
- net DLEFT_5: now also U30.16 (B6)
- net DLEFT_6: now also U30.15 (B7)
- net DLEFT_7: now also U30.14 (B8)
- net GND: now also C44.1, C45.1, U30.11 (GND), U30.12 (GND), U30.13 (GND), U30.22 (~OE), U32.14 (2~OE), U32.15 (1~OE), U32.7 (2A2), U32.8 (GND), U32.9 (GND)
- net OPC_CLK: now also U32.6 (2A1); no longer IC1.22 (P22/GCK0)
- net OPLEFT_CLK: now also U32.4 (1A1); no longer IC1.27 (P27/GCLK2)
- net OPRIGHT_CLK: now also U32.5 (1A2); no longer IC1.23 (P23/GCK1)
- new net CPLD_OPC_CLK: IC1.22 (P22/GCK0), U32.11 (2B1)
- new net CPLD_OPLEFT_CLK: IC1.27 (P27/GCLK2), U32.13 (1B1)
- new net CPLD_OPRIGHT_CLK: IC1.23 (P23/GCK1), U32.12 (1B2)
- new net NUMBER_0: U30.3 (A1)
- new net NUMBER_1: U30.4 (A2)
- new net NUMBER_2: U30.5 (A3)
- new net NUMBER_3: U30.6 (A4)
- new net NUMBER_4: U30.7 (A5)
- new net NUMBER_5: U30.8 (A6)
- new net NUMBER_6: U30.9 (A7)
- new net NUMBER_7: U30.10 (A8)
- no-connect marks 17 -> 18
Other:
- moved on the sheet: C33, C40, U28

Commit message: Renaming files, cleaning, CHANGELOG
Connections:
- net CPLD_OPLEFT_CLK: now also J5.34 (Pin_34)
- net CPLD_OPRIGHT_CLK: now also J5.36 (Pin_36)
- net GND: no longer U32.7 (2A2)
- net OPLEFT_CLK: no longer J5.34 (Pin_34)
- net OPRIGHT_CLK: no longer J5.36 (Pin_36)
- net CPLD_OPC_CLK renamed CPLD_OPCHOOSE_CLK
- net CPLD_OPCHOOSE_CLK: now also J5.35 (Pin_35)
- net OPC_CLK renamed OPCHOOSE_CLK
- net OPCHOOSE_CLK: now also U32.7 (2A2); no longer J5.35 (Pin_35)
Other:
- moved on the sheet: C44, U32
Changed lines of the file:
@@
 $EndComp
 Text HLabel 1300 1950 0    60   Input ~ 0
-OPC_CLK
+OPCHOOSE_CLK
 Text HLabel 1300 1750 0    60   Input ~ 0
 OPLEFT_CLK
@@
 Wire Bus Line
 	1400 1550 1300 1550
-Text Label 2100 5950 0    60   ~ 0
+Text Label 2400 5950 0    60   ~ 0
 CPLD_OPLEFT_CLK
-Text Label 2100 6050 0    60   ~ 0
+Text Label 2400 6050 0    60   ~ 0
 CPLD_OPRIGHT_CLK
-Text Label 2100 6150 0    60   ~ 0
-CPLD_OPC_CLK
+Text Label 2400 6150 0    60   ~ 0
+CPLD_OPCHOOSE_CLK
 $Comp
 L power:GND #PWR012
@@
 Text Label 10450 3350 0    60   ~ 0
 OPCS_7
-Text Label 9950 2550 2    60   ~ 0
-OPLEFT_CLK
-Text Label 9950 2450 2    60   ~ 0
-OPRIGHT_CLK
-Text Label 10450 2450 0    60   ~ 0
-OPC_CLK
 Text Label 9950 3350 2    60   ~ 0
 DRIGHT_0
@@
 L Custom:SN74AVC4T245D U32
 U 1 1 5EF08705
-P 1600 5850
-F 0 "U32" H 1800 6500 50  0000 C CNN
-F 1 "SN74AVC4T245D" H 2050 6400 50  0000 C CNN
-F 2 "" H 1600 5750 50  0001 C CNN
-F 3 "http://www.ti.com/lit/ds/symlink/sn74avc4t245.pdf" H 1550 5600 50  0001 C CNN
-	1    1600 5850
-	1    0    0    -1
-$EndComp
-Text Label 1100 5950 2    60   ~ 0
+P 1900 5850
+F 0 "U32" H 2100 6500 50  0000 C CNN
+F 1 "SN74AVC4T245D" H 2350 6400 50  0000 C CNN
+F 2 "" H 1900 5750 50  0001 C CNN
+F 3 "http://www.ti.com/lit/ds/symlink/sn74avc4t245.pdf" H 1850 5600 50  0001 C CNN
+	1    1900 5850
+	1    0    0    -1
+$EndComp
+Text Label 1400 5950 2    60   ~ 0
 OPLEFT_CLK
-Text Label 1100 6050 2    60   ~ 0
+Text Label 1400 6050 2    60   ~ 0
 OPRIGHT_CLK
-Text Label 1100 6150 2    60   ~ 0
-OPC_CLK
+Text Label 1400 6150 2    60   ~ 0
+OPCHOOSE_CLK
 Text Label 1350 1750 0    60   ~ 0
 OPLEFT_CLK
@@
 OPRIGHT_CLK
 Text Label 1350 1950 0    60   ~ 0
-OPC_CLK
+OPCHOOSE_CLK
 $Comp
 L power:+3.3V #PWR037
 U 1 1 5EF5FE0F
-P 1600 5150
-F 0 "#PWR037" H 1600 5000 50  0001 C CNN
-F 1 "+3.3V" H 1600 5290 50  0000 C CNN
-F 2 "" H 1600 5150 50  0001 C CNN
-F 3 "" H 1600 5150 50  0001 C CNN
-	1    1600 5150
-	1    0    0    -1
-$EndComp
-Wire Wire Line
-	1700 5250 1700 5200
-Wire Wire Line
-	1700 5200 1600 5200
-Wire Wire Line
-	1600 5200 1600 5150
-Wire Wire Line
-	1600 5200 1500 5200
-Wire Wire Line
-	1500 5200 1500 5250
-Connection ~ 1600 5200
+P 1900 5150
+F 0 "#PWR037" H 1900 5000 50  0001 C CNN
+F 1 "+3.3V" H 1900 5290 50  0000 C CNN
+F 2 "" H 1900 5150 50  0001 C CNN
+F 3 "" H 1900 5150 50  0001 C CNN
+	1    1900 5150
+	1    0    0    -1
+$EndComp
+Wire Wire Line
+	2000 5250 2000 5200
+Wire Wire Line
+	2000 5200 1900 5200
+Wire Wire Line
+	1900 5200 1900 5150
+Wire Wire Line
+	1900 5200 1800 5200
+Wire Wire Line
+	1800 5200 1800 5250
+Connection ~ 1900 5200
 $Comp
 L Device:C C?
 U 1 1 5EF7425E
-P 850 5200
+P 1150 5200
 AR Path="/5EF7425E" Ref="C?"  Part="1"
 AR Path="/5AA18AD6/5EF7425E" Ref="C44"  Part="1"
-F 0 "C44" H 875 5300 50  0000 L CNN
-F 1 "10nF" H 875 5100 50  0000 L CNN
-F 2 "Capacitor_SMD:C_0805_2012Metric" H 888 5050 50  0001 C CNN
-F 3 "" H 850 5200 50  0001 C CNN
-	1    850  5200
+F 0 "C44" H 1175 5300 50  0000 L CNN
+F 1 "10nF" H 1175 5100 50  0000 L CNN
+F 2 "Capacitor_SMD:C_0805_2012Metric" H 1188 5050 50  0001 C CNN
+F 3 "" H 1150 5200 50  0001 C CNN
+	1    1150 5200
 	0    -1   -1   0
 $EndComp
 Wire Wire Line
-	1100 5750 1050 5750
-Wire Wire Line
-	1050 5750 1050 5650
-Wire Wire Line
-	1050 5200 1000 5200
-Wire Wire Line
-	1100 5650 1050 5650
-Connection ~ 1050 5650
-Wire Wire Line
-	1050 5650 1050 5200
-Wire Wire Line
-	1050 5200 1500 5200
-Connection ~ 1050 5200
-Connection ~ 1500 5200
-Wire Wire Line
-	1100 6250 1050 6250
-Wire Wire Line
-	1050 6250 1050 6500
-Wire Wire Line
-	1050 6500 1600 6500
-Wire Wire Line
-	1600 6500 1600 6450
+	1400 5750 1350 5750
+Wire Wire Line
+	1350 5750 1350 5650
+Wire Wire Line
+	1350 5200 1300 5200
+Wire Wire Line
+	1400 5650 1350 5650
+Connection ~ 1350 5650
+Wire Wire Line
+	1350 5650 1350 5200
+Wire Wire Line
+	1350 5200 1800 5200
+Connection ~ 1350 5200
+Connection ~ 1800 5200
+Wire Wire Line
+	1900 6500 1900 6450
 $Comp
 L power:GND #PWR038
 U 1 1 5EFAB461
-P 1600 6550
-F 0 "#PWR038" H 1600 6300 50  0001 C CNN
-F 1 "GND" H 1605 6377 50  0000 C CNN
-F 2 "" H 1600 6550 50  0001 C CNN
-F 3 "" H 1600 6550 50  0001 C CNN
-	1    1600 6550
-	1    0    0    -1
-$EndComp
-Wire Wire Line
-	1600 6550 1600 6500
-Connection ~ 1600 6500
-Wire Wire Line
-	1050 6500 500  6500
-Wire Wire Line
-	500  6500 500  5550
-Wire Wire Line
-	500  5200 700  5200
-Connection ~ 1050 6500
-Wire Wire Line
-	1100 5450 500  5450
-Connection ~ 500  5450
-Wire Wire Line
-	500  5450 500  5200
-Wire Wire Line
-	1100 5550 500  5550
-Connection ~ 500  5550
-Wire Wire Line
-	500  5550 500  5450
-NoConn ~ 2100 6250
+P 1900 6550
+F 0 "#PWR038" H 1900 6300 50  0001 C CNN
+F 1 "GND" H 1905 6377 50  0000 C CNN
+F 2 "" H 1900 6550 50  0001 C CNN
+F 3 "" H 1900 6550 50  0001 C CNN
+	1    1900 6550
+	1    0    0    -1
+$EndComp
+Wire Wire Line
+	1900 6550 1900 6500
+Connection ~ 1900 6500
+NoConn ~ 2400 6250
 Text Label 4050 4200 2    60   ~ 0
 CPLD_OPLEFT_CLK
 Text Label 4050 3950 2    60   ~ 0
 CPLD_OPRIGHT_CLK
+Wire Wire Line
+	700  6500 700  5550
+Wire Wire Line
+	700  5200 1000 5200
+Connection ~ 700  5450
+Wire Wire Line
+	700  5450 700  5200
+Wire Wire Line
+	700  5450 1400 5450
+Wire Wire Line
+	700  5550 1400 5550
+Connection ~ 700  5550
+Wire Wire Line
+	700  5550 700  5450
 Text Label 4050 3850 2    60   ~ 0
-CPLD_OPC_CLK
+CPLD_OPCHOOSE_CLK
+Text Label 10450 2450 0    60   ~ 0
+CPLD_OPCHOOSE_CLK
+Text Label 9950 2450 2    60   ~ 0
+CPLD_OPRIGHT_CLK
+Text Label 9950 2550 2    60   ~ 0
+CPLD_OPLEFT_CLK
+Wire Wire Line
+	700  6500 1900 6500
+Text Label 1400 6250 2    60   ~ 0
+OPCHOOSE_CLK
 Wire Bus Line
 	1400 750  1400 1550

Commit message: Cleaning
Parts:
- IC1: footprint (none) -> Package_QFP:VQFP-100_14x14mm_P0.5mm
- J1: footprint (none) -> Connector_PinSocket_2.54mm:PinSocket_1x06_P2.54mm_Vertical
- J4: footprint (none) -> Connector_PinHeader_1.27mm:PinHeader_2x15_P1.27mm_Vertical
- J5: footprint (none) -> Connector_PinHeader_1.27mm:PinHeader_2x19_P1.27mm_Vertical
- U28: footprint (none) -> Package_TO_SOT_SMD:SOT-23
- U30: footprint (none) -> Package_SO:SOIC-24W_7.5x15.4mm_P1.27mm
- U32: footprint (none) -> Package_SO:SOIC-16_3.9x9.9mm_P1.27mm
Changed lines of the file:
@@
 F 0 "IC1" H 5700 6250 50  0000 C CNN
 F 1 "XC2C256-VQ100" H 4300 6250 50  0000 C CNN
-F 2 "" H 5200 3800 50  0001 C CNN
+F 2 "Package_QFP:VQFP-100_14x14mm_P0.5mm" H 5200 3800 50  0001 C CNN
 F 3 "" H 5200 3800 50  0001 C CNN
 	1    5200 3800
@@
 F 0 "J4" H 8500 2525 50  0000 C CNN
 F 1 "UnusedPins_Connector" H 8500 2616 50  0000 C CNN
-F 2 "" H 8450 3450 50  0001 C CNN
+F 2 "Connector_PinHeader_1.27mm:PinHeader_2x15_P1.27mm_Vertical" H 8450 3450 50  0001 C CNN
 F 3 "~" H 8450 3450 50  0001 C CNN
 	1    8450 3450
@@
 F 0 "J5" H 10300 2125 50  0000 C CNN
 F 1 "ALU_PINS" H 10300 2216 50  0000 C CNN
-F 2 "" H 10250 3250 50  0001 C CNN
+F 2 "Connector_PinHeader_1.27mm:PinHeader_2x19_P1.27mm_Vertical" H 10250 3250 50  0001 C CNN
 F 3 "~" H 10250 3250 50  0001 C CNN
 	1    10250 3250
@@
 F 0 "J1" H 8272 1232 50  0000 R CNN
 F 1 "ALU_JTAG" H 8272 1323 50  0000 R CNN
-F 2 "" H 8300 1350 50  0001 C CNN
+F 2 "Connector_PinSocket_2.54mm:PinSocket_1x06_P2.54mm_Vertical" H 8300 1350 50  0001 C CNN
 F 3 "~" H 8300 1350 50  0001 C CNN
 	1    8300 1350
@@
 F 0 "U28" H 3400 7092 50  0000 C CNN
 F 1 "TPS7A0518PDBZR" H 3400 7001 50  0000 C CNN
-F 2 "" H 3400 6750 50  0001 C CNN
+F 2 "Package_TO_SOT_SMD:SOT-23" H 3400 6750 50  0001 C CNN
 F 3 "" H 3400 6750 50  0001 C CNN
 	1    3400 6850
@@
 F 0 "U30" H 1850 3600 50  0000 C CNN
 F 1 "SN74LVC8T245DW" H 2100 3500 50  0000 C CNN
-F 2 "" H 2500 2300 50  0001 C CNN
+F 2 "Package_SO:SOIC-24W_7.5x15.4mm_P1.27mm" H 2500 2300 50  0001 C CNN
 F 3 "http://www.ti.com/lit/ds/symlink/sn74lvc8t245.pdf" H 1550 2700 50  0001 C CNN
 	1    1600 2950
@@
 F 0 "U32" H 2100 6500 50  0000 C CNN
 F 1 "SN74AVC4T245D" H 2350 6400 50  0000 C CNN
-F 2 "" H 1900 5750 50  0001 C CNN
+F 2 "Package_SO:SOIC-16_3.9x9.9mm_P1.27mm" H 1900 5750 50  0001 C CNN
 F 3 "http://www.ti.com/lit/ds/symlink/sn74avc4t245.pdf" H 1850 5600 50  0001 C CNN
 	1    1900 5850
