File: fileOperation.sch (KiCad schematic (older format))
At the start: 19 parts, among them IC1 XC2C256-VQ100, J1 ALU_JTAG, J4 UnusedPins_Connector, J5 ALU_PINS, U28 TPS7A0518PDBZR, U30 SN74LVC8T245DW, U32 SN74AVC4T245D

Commit message: V5.1 (#9)
* Apply new symbol for XC2C256-VQ100 #5

* Set new date and 5.1

* Replacing 74HC165 with 74HC166, and add SPI_CFG_DS #4

* Replace some gates with a 74AHC1G02 to fix the pulse problem #3

* Go next only if SRCVALUE, (simple instruction)

* Remove weird ghost bus in register

* Small cleaning in fileRegister

* Go next only if SRCVALUE, (complex instruction) #8
adding 74AHC1G08

* Better decoupling #6

* Component association (#7)

* netlist

* Updated BOM for V5.1

* Routing, cleaning first pass

* bit of pcb cleaning

* SolderMaskClearance to 0

* Schematics to pdf

* PCB files in pdf

* exporting Gerbert files

* new 3d images

* Update README.md

* Modifying CHANGELOG file

* Update README.md
Parts:
- J1: footprint Connector_PinSocket_2.54mm:PinSocket_1x06_P2.54mm_Vertical -> Connector_PinHeader_2.54mm:PinHeader_1x06_P2.54mm_Vertical
Connections:
- wire segments 196 -> 180
