File: fileNumberSelect.sch (KiCad schematic (older format))
At the start: 13 parts, among them U17 74AHC138, U19 74AHCT244, U20 74AHCT244, U21 74AHCT244, U22 74AHCT244, U23 74AHCT244

Commit message: Go next only if SRCVALUE, (simple instruction)
Changed lines of the file:
@@
 Text Label 10200 2100 2    60   ~ 0
 ~SELECTING_SPI
+Text Label 10200 1750 2    60   ~ 0
+~SELECTING_SRC
+Text HLabel 10250 1750 2    60   Output ~ 0
+~SELECTING_SRC
+Wire Wire Line
+	10200 1750 10250 1750
 Wire Bus Line
 	9500 800  9500 1550
