File: fileNumberSelect.sch (KiCad schematic (older format))
At the start: 13 parts, among them U17 74AHC138, U19 74AHCT244, U20 74AHCT244, U21 74AHCT244, U22 74AHCT244, U23 74AHCT244

Commit message: V5.1 (#9)
* Apply new symbol for XC2C256-VQ100 #5

* Set new date and 5.1

* Replacing 74HC165 with 74HC166, and add SPI_CFG_DS #4

* Replace some gates with a 74AHC1G02 to fix the pulse problem #3

* Go next only if SRCVALUE, (simple instruction)

* Remove weird ghost bus in register

* Small cleaning in fileRegister

* Go next only if SRCVALUE, (complex instruction) #8
adding 74AHC1G08

* Better decoupling #6

* Component association (#7)

* netlist

* Updated BOM for V5.1

* Routing, cleaning first pass

* bit of pcb cleaning

* SolderMaskClearance to 0

* Schematics to pdf

* PCB files in pdf

* exporting Gerbert files

* new 3d images

* Update README.md

* Modifying CHANGELOG file

* Update README.md
Changed lines of the file:
@@
 Sheet 3 8
 Title "GP8B"
-Date "2020-08-19"
-Rev "V5.0"
+Date "2021-03-04"
+Rev "V5.1"
 Comp "Guillaume Guillet"
-Comment1 "Copyright Guillaume Guillet 2020"
+Comment1 "Copyright Guillaume Guillet 2021"
 Comment2 "Licensed under CERN-OHL-W v2 or later"
 Comment3 ""
@@
 Text Label 10200 2100 2    60   ~ 0
 ~SELECTING_SPI
+Text Label 10200 1750 2    60   ~ 0
+~SELECTING_SRC
+Text HLabel 10250 1750 2    60   Output ~ 0
+~SELECTING_SRC
+Wire Wire Line
+	10200 1750 10250 1750
 Wire Bus Line
 	9500 800  9500 1550
