File: Project_GP8B.kicad_pcb (KiCad board)
At the start: 4 copper layers, 133 x 93 mm, 110 parts, among them IC1 XC2C256-VQ100, J1 ALU_JTAG, J2 TE_Eurocard_96pole, J3 MM1_5530843-2, J4 UnusedPins_Connector, J5 ALU_PINS, U1 74AHC05, U10 74AHC1G04, U11 CD74AC238, U12 74AHC1G04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

Commit message: SolderMaskClearance to 0
Other:
- rule pad_to_mask_clearance: 0.2 -> 0
