File: fileSPI.kicad_sch (KiCad schematic)
At the start: 6 parts

Commit message: Updating descriptions
Parts:
- C41, C42, C43: renamed from C?; value (none) -> 10nF; footprint (none) -> Capacitor_SMD:C_0805_2012Metric
- U18: value (none) -> 74HC166; footprint (none) -> Package_SO:SOIC-16_3.9x9.9mm_P1.27mm
- U25: value (none) -> 74AHCT595; footprint (none) -> Package_SO:SOIC-16_3.9x9.9mm_P1.27mm
- U6: renamed from U?; value (none) -> 74AHC273; footprint (none) -> Package_SO:SOIC-20W_7.5x12.8mm_P1.27mm
Changed lines of the file:
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@@
   (title_block
     (title "GP8B")
-    (date "2021-03-04")
-    (rev "V5.1")
+    (date "2022-07-08")
+    (rev "V6.0")
     (company "Guillaume Guillet")
-    (comment 1 "Copyright Guillaume Guillet 2021")
+    (comment 1 "Copyright Guillaume Guillet 2022")
     (comment 2 "Licensed under CERN-OHL-W v2 or later")
   )
@@
     (in_bom yes) (on_board yes)
     (property "Reference" "U25" (id 0) (at 204.47 52.07 0))
-    (property "Value" "" (id 1) (at 208.28 54.61 0))
-    (property "Footprint" "" (id 2) (at 200.66 68.58 0)
+    (property "Value" "74AHCT595" (id 1) (at 208.28 54.61 0))
+    (property "Footprint" "Package_SO:SOIC-16_3.9x9.9mm_P1.27mm" (id 2) (at 200.66 68.58 0)
       (effects (font (size 1.27 1.27)) hide)
     )
@@
   (symbol (lib_id "power:+5V") (at 80.01 48.26 0) (unit 1)
     (in_bom yes) (on_board yes)
-    (property "Reference" "#PWR?" (id 0) (at 80.01 52.07 0)
-      (effects (font (size 1.27 1.27)) hide)
-    )
-    (property "Value" "" (id 1) (at 80.01 44.704 0))
+    (property "Reference" "#PWR0133" (id 0) (at 80.01 52.07 0)
+      (effects (font (size 1.27 1.27)) hide)
+    )
+    (property "Value" "+5V" (id 1) (at 80.01 44.704 0))
     (property "Footprint" "" (id 2) (at 80.01 48.26 0)
       (effects (font (size 1.27 1.27)) hide)
@@
   (symbol (lib_id "power:GND") (at 80.01 93.98 0) (unit 1)
     (in_bom yes) (on_board yes)
-    (property "Reference" "#PWR?" (id 0) (at 80.01 100.33 0)
-      (effects (font (size 1.27 1.27)) hide)
-    )
-    (property "Value" "" (id 1) (at 80.01 97.79 0))
+    (property "Reference" "#PWR0134" (id 0) (at 80.01 100.33 0)
+      (effects (font (size 1.27 1.27)) hide)
+    )
+    (property "Value" "GND" (id 1) (at 80.01 97.79 0))
     (property "Footprint" "" (id 2) (at 80.01 93.98 0)
       (effects (font (size 1.27 1.27)) hide)
@@
   (symbol (lib_id "Device:C") (at 49.53 88.9 180) (unit 1)
     (in_bom yes) (on_board yes)
-    (property "Reference" "C?" (id 0) (at 48.895 91.44 0)
-      (effects (font (size 1.27 1.27)) (justify left))
-    )
-    (property "Value" "" (id 1) (at 48.895 86.36 0)
-      (effects (font (size 1.27 1.27)) (justify left))
-    )
-    (property "Footprint" "" (id 2) (at 48.5648 85.09 0)
+    (property "Reference" "C41" (id 0) (at 48.895 91.44 0)
+      (effects (font (size 1.27 1.27)) (justify left))
+    )
+    (property "Value" "10nF" (id 1) (at 48.895 86.36 0)
+      (effects (font (size 1.27 1.27)) (justify left))
+    )
+    (property "Footprint" "Capacitor_SMD:C_0805_2012Metric" (id 2) (at 48.5648 85.09 0)
       (effects (font (size 1.27 1.27)) hide)
     )
@@
   (symbol (lib_id "74xx:74AHC273") (at 80.01 71.12 0) (unit 1)
     (in_bom yes) (on_board yes)
-    (property "Reference" "U?" (id 0) (at 83.82 52.07 0))
-    (property "Value" "" (id 1) (at 86.36 54.61 0))
-    (property "Footprint" "" (id 2) (at 80.01 71.12 0)
+    (property "Reference" "U6" (id 0) (at 83.82 52.07 0))
+    (property "Value" "74AHC273" (id 1) (at 86.36 54.61 0))
+    (property "Footprint" "Package_SO:SOIC-20W_7.5x12.8mm_P1.27mm" (id 2) (at 80.01 71.12 0)
       (effects (font (size 1.27 1.27)) hide)
     )
@@
   (symbol (lib_id "power:+5V") (at 143.51 44.45 0) (unit 1)
     (in_bom yes) (on_board yes)
-    (property "Reference" "#PWR?" (id 0) (at 143.51 48.26 0)
-      (effects (font (size 1.27 1.27)) hide)
-    )
-    (property "Value" "" (id 1) (at 143.51 40.894 0))
+    (property "Reference" "#PWR0135" (id 0) (at 143.51 48.26 0)
+      (effects (font (size 1.27 1.27)) hide)
+    )
+    (property "Value" "+5V" (id 1) (at 143.51 40.894 0))
     (property "Footprint" "" (id 2) (at 143.51 44.45 0)
       (effects (font (size 1.27 1.27)) hide)
@@
   (symbol (lib_id "power:GND") (at 143.51 100.33 0) (unit 1)
     (in_bom yes) (on_board yes)
-    (property "Reference" "#PWR?" (id 0) (at 143.51 106.68 0)
-      (effects (font (size 1.27 1.27)) hide)
-    )
-    (property "Value" "" (id 1) (at 143.51 104.14 0))
+    (property "Reference" "#PWR0136" (id 0) (at 143.51 106.68 0)
+      (effects (font (size 1.27 1.27)) hide)
+    )
+    (property "Value" "GND" (id 1) (at 143.51 104.14 0))
     (property "Footprint" "" (id 2) (at 143.51 100.33 0)
       (effects (font (size 1.27 1.27)) hide)
@@
   (symbol (lib_id "power:GND") (at 200.66 88.9 0) (unit 1)
     (in_bom yes) (on_board yes)
-    (property "Reference" "#PWR?" (id 0) (at 200.66 95.25 0)
-      (effects (font (size 1.27 1.27)) hide)
-    )
-    (property "Value" "" (id 1) (at 200.66 92.71 0))
+    (property "Reference" "#PWR0137" (id 0) (at 200.66 95.25 0)
+      (effects (font (size 1.27 1.27)) hide)
+    )
+    (property "Value" "GND" (id 1) (at 200.66 92.71 0))
     (property "Footprint" "" (id 2) (at 200.66 88.9 0)
       (effects (font (size 1.27 1.27)) hide)
@@
   (symbol (lib_id "power:+5V") (at 200.66 50.8 0) (unit 1)
     (in_bom yes) (on_board yes)
-    (property "Reference" "#PWR?" (id 0) (at 200.66 54.61 0)
-      (effects (font (size 1.27 1.27)) hide)
-    )
-    (property "Value" "" (id 1) (at 200.66 47.244 0))
+    (property "Reference" "#PWR0138" (id 0) (at 200.66 54.61 0)
+      (effects (font (size 1.27 1.27)) hide)
+    )
+    (property "Value" "+5V" (id 1) (at 200.66 47.244 0))
     (property "Footprint" "" (id 2) (at 200.66 50.8 0)
       (effects (font (size 1.27 1.27)) hide)
@@
   (symbol (lib_id "Device:C") (at 115.57 92.71 180) (unit 1)
     (in_bom yes) (on_board yes)
-    (property "Reference" "C?" (id 0) (at 114.935 95.25 0)
-      (effects (font (size 1.27 1.27)) (justify left))
-    )
-    (property "Value" "" (id 1) (at 114.935 90.17 0)
-      (effects (font (size 1.27 1.27)) (justify left))
-    )
-    (property "Footprint" "" (id 2) (at 114.6048 88.9 0)
+    (property "Reference" "C42" (id 0) (at 114.935 95.25 0)
+      (effects (font (size 1.27 1.27)) (justify left))
+    )
+    (property "Value" "10nF" (id 1) (at 114.935 90.17 0)
+      (effects (font (size 1.27 1.27)) (justify left))
+    )
+    (property "Footprint" "Capacitor_SMD:C_0805_2012Metric" (id 2) (at 114.6048 88.9 0)
       (effects (font (size 1.27 1.27)) hide)
     )
@@
   (symbol (lib_id "Device:C") (at 172.72 83.82 180) (unit 1)
     (in_bom yes) (on_board yes)
-    (property "Reference" "C?" (id 0) (at 172.085 86.36 0)
-      (effects (font (size 1.27 1.27)) (justify left))
-    )
-    (property "Value" "" (id 1) (at 172.085 81.28 0)
-      (effects (font (size 1.27 1.27)) (justify left))
-    )
-    (property "Footprint" "" (id 2) (at 171.7548 80.01 0)
+    (property "Reference" "C43" (id 0) (at 172.085 86.36 0)
+      (effects (font (size 1.27 1.27)) (justify left))
+    )
+    (property "Value" "10nF" (id 1) (at 172.085 81.28 0)
+      (effects (font (size 1.27 1.27)) (justify left))
+    )
+    (property "Footprint" "Capacitor_SMD:C_0805_2012Metric" (id 2) (at 171.7548 80.01 0)
       (effects (font (size 1.27 1.27)) hide)
     )
@@
       (effects (font (size 1.27 1.27)) (justify left))
     )
-    (property "Value" "" (id 1) (at 146.05 50.8 0)
-      (effects (font (size 1.27 1.27)) (justify left))
-    )
-    (property "Footprint" "" (id 2) (at 143.51 72.39 0)
-      (effects (font (size 1.27 1.27)) hide)
-    )
+    (property "Value" "74HC166" (id 1) (at 146.05 50.8 0)
+      (effects (font (size 1.27 1.27)) (justify left))
+    )
+    (property "Footprint" "Package_SO:SOIC-16_3.9x9.9mm_P1.27mm" (id 2) (at 143.51 72.39 0)
+      (effects (font (size 1.27 1.27)) hide)
+    )
