File: fileSPI.kicad_sch (KiCad schematic)
At the start: 6 parts, among them U18 74HC166, U25 74AHCT595, U6 74AHC273

Commit message: update BOM
Parts:
- U6: footprint Package_SO:SOIC-20W_7.5x12.8mm_P1.27mm -> Package_SO:SSOP-20_5.3x7.2mm_P0.65mm
Changed lines of the file:
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@@
       (effects (font (size 1.27 1.27)))
     )
-    (property "Footprint" "Package_SO:SOIC-20W_7.5x12.8mm_P1.27mm" (at 80.01 71.12 0)
+    (property "Footprint" "Package_SO:SSOP-20_5.3x7.2mm_P0.65mm" (at 80.01 71.12 0)
       (effects (font (size 1.27 1.27)) hide)
     )
