File: fileOperation.kicad_sch (KiCad schematic)
At the start: 19 parts

Commit message: Updating descriptions
Parts:
- C20, C24, C26, C28, C32, C39, C7, C9: value (none) -> 100nF; footprint (none) -> Capacitor_SMD:C_0805_2012Metric
- C33, C40: value (none) -> 1uF; footprint (none) -> Capacitor_SMD:C_0805_2012Metric
- C44, C45: renamed from C?; value (none) -> 10nF; footprint (none) -> Capacitor_SMD:C_0805_2012Metric
- IC1: value (none) -> XC2C256-VQ100; footprint (none) -> Package_QFP:VQFP-100_14x14mm_P0.5mm
- J1: value (none) -> ALU_JTAG; footprint (none) -> Connector_PinHeader_2.54mm:PinHeader_1x06_P2.54mm_Vertical
- J4: value (none) -> UnusedPins_Connector; footprint (none) -> Connector_PinHeader_1.27mm:PinHeader_2x15_P1.27mm_Vertical
- J5: value (none) -> ALU_PINS; footprint (none) -> Connector_PinHeader_1.27mm:PinHeader_2x19_P1.27mm_Vertical
- U28: value (none) -> TPS7A0518PDBZR; footprint (none) -> Package_TO_SOT_SMD:SOT-23
- U30: value (none) -> SN74LVC8T245DW; footprint (none) -> Package_SO:SOIC-24W_7.5x15.4mm_P1.27mm
- U32: value (none) -> SN74AVC4T245D; footprint (none) -> Package_SO:SOIC-16_3.9x9.9mm_P1.27mm
