File: fileOperation.kicad_sch (KiCad schematic)
At the start: 19 parts, among them IC1 XC2C256-VQ100, J1 ALU_JTAG, J4 UnusedPins_Connector, J5 ALU_PINS, U28 TPS7A0518PDBZR, U30 SN74LVC8T245DW, U32 SN74AVC4T245D

Commit message: updating symbols ref, renaming some pins (NEXT_AFTERSET -> REQ_NEXT_AFTERISET)
Parts:
- J1: symbol Connector:Conn_01x06_Male -> Connector:Conn_01x06_Pin
Changed lines of the file:
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@@
       (effects (font (size 1.27 1.27)) hide)
     )
-    (property "Datasheet" "" (at 132.08 96.52 0)
+    (property "Datasheet" "https://www.xilinx.com/support/documentation/data_sheets/ds094.pdf" (at 132.08 96.52 0)
       (effects (font (size 1.27 1.27)) hide)
     )
@@
       (effects (font (size 1.27 1.27)) hide)
     )
-    (property "Datasheet" "" (at 22.86 58.42 0)
+    (property "Datasheet" "~" (at 22.86 58.42 0)
       (effects (font (size 1.27 1.27)) hide)
     )
@@
       (effects (font (size 1.27 1.27)) hide)
     )
-    (property "Datasheet" "" (at 29.21 132.08 0)
+    (property "Datasheet" "~" (at 29.21 132.08 0)
       (effects (font (size 1.27 1.27)) hide)
     )
@@
     )
   )
-  (symbol (lib_id "Connector:Conn_01x06_Male") (at 210.82 34.29 180) (unit 1)
+  (symbol (lib_id "Connector:Conn_01x06_Pin") (at 210.82 34.29 180) (unit 1)
     (in_bom yes) (on_board yes) (dnp no)
     (property "Reference" "J1" (at 211.5312 31.2928 0)

Commit message: update BOM
Parts:
- U30: footprint Package_SO:SOIC-24W_7.5x15.4mm_P1.27mm -> Package_SO:SSOP-24_5.3x8.2mm_P0.65mm
Changed lines of the file:
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@@
       (effects (font (size 1.27 1.27)))
     )
-    (property "Footprint" "Package_SO:SOIC-24W_7.5x15.4mm_P1.27mm" (at 63.5 91.44 0)
+    (property "Footprint" "Package_SO:SSOP-24_5.3x8.2mm_P0.65mm" (at 63.5 91.44 0)
       (effects (font (size 1.27 1.27)) hide)
     )
