File: Project_GP8B.kicad_sch (KiCad schematic)
At the start: 15 parts, among them U1 74AHC05, U2 74AHC05, U5 74AHC05

Commit message: updating symbols ref, renaming some pins (NEXT_AFTERSET -> REQ_NEXT_AFTERISET)
Connections:
- net END_ISIMPLE renamed REQ_END_ISIMPLE
- net END_MAXCOUNT renamed REQ_END_MAXSEQ
- net NEXT_AFTERSET renamed REQ_NEXT_AFTERISET
- net NEXT_ISIMPLE renamed REQ_NEXT_ISIMPLE
Other:
- sheet Instruction ports: added REQ_END_ISIMPLE, REQ_END_MAXSEQ, REQ_NEXT_AFTERISET, REQ_NEXT_ISIMPLE; removed END_ISIMPLE, END_MAXCOUNT, NEXT_AFTERSET, NEXT_ISIMPLE
Changed lines of the file:
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@@
     (effects (font (size 1.524 1.524)) (justify right bottom))
   )
-  (label "END_ISIMPLE" (at 35.56 125.73 180) (fields_autoplaced)
+  (label "REQ_END_ISIMPLE" (at 35.56 125.73 180) (fields_autoplaced)
     (effects (font (size 1.524 1.524)) (justify right bottom))
   )
@@
     (effects (font (size 1.524 1.524)) (justify left bottom))
   )
-  (label "NEXT_AFTERSET" (at 113.03 144.78 180) (fields_autoplaced)
+  (label "REQ_NEXT_AFTERISET" (at 113.03 144.78 180) (fields_autoplaced)
     (effects (font (size 1.524 1.524)) (justify right bottom))
   )
@@
     (effects (font (size 1.524 1.524)) (justify right bottom))
   )
-  (label "END_ISIMPLE" (at 261.62 92.71 0) (fields_autoplaced)
+  (label "REQ_END_ISIMPLE" (at 261.62 92.71 0) (fields_autoplaced)
     (effects (font (size 1.524 1.524)) (justify left bottom))
   )
@@
     (effects (font (size 1.524 1.524)) (justify right bottom))
   )
-  (label "END_MAXCOUNT" (at 35.56 130.81 180) (fields_autoplaced)
+  (label "REQ_END_MAXSEQ" (at 35.56 130.81 180) (fields_autoplaced)
     (effects (font (size 1.524 1.524)) (justify right bottom))
   )
@@
     (effects (font (size 1.524 1.524)) (justify left bottom))
   )
-  (label "NEXT_AFTERSET" (at 261.62 87.63 0) (fields_autoplaced)
+  (label "REQ_NEXT_AFTERISET" (at 261.62 87.63 0) (fields_autoplaced)
     (effects (font (size 1.524 1.524)) (justify left bottom))
   )
@@
     (effects (font (size 1.524 1.524)) (justify left bottom))
   )
-  (label "NEXT_ISIMPLE" (at 261.62 95.25 0) (fields_autoplaced)
+  (label "REQ_NEXT_ISIMPLE" (at 261.62 95.25 0) (fields_autoplaced)
     (effects (font (size 1.524 1.524)) (justify left bottom))
   )
@@
     (effects (font (size 1.524 1.524)) (justify right bottom))
   )
-  (label "END_MAXCOUNT" (at 261.62 90.17 0) (fields_autoplaced)
+  (label "REQ_END_MAXSEQ" (at 261.62 90.17 0) (fields_autoplaced)
     (effects (font (size 1.524 1.524)) (justify left bottom))
   )
@@
     (effects (font (size 1.524 1.524)) (justify right bottom))
   )
-  (label "NEXT_ISIMPLE" (at 113.03 142.24 180) (fields_autoplaced)
+  (label "REQ_NEXT_ISIMPLE" (at 113.03 142.24 180) (fields_autoplaced)
     (effects (font (size 1.524 1.524)) (justify right bottom))
   )
@@
       (effects (font (size 1.27 1.27)) hide)
     )
-    (property "Datasheet" "" (at 118.11 133.35 0)
+    (property "Datasheet" "~" (at 118.11 133.35 0)
       (effects (font (size 1.27 1.27)) hide)
     )
@@
       (effects (font (size 1.27 1.27)) hide)
     )
-    (property "Datasheet" "" (at 140.97 137.16 0)
+    (property "Datasheet" "~" (at 140.97 137.16 0)
       (effects (font (size 1.27 1.27)) hide)
     )
@@
       (effects (font (size 1.27 1.27)) hide)
     )
-    (property "Datasheet" "" (at 40.64 158.75 0)
+    (property "Datasheet" "~" (at 40.64 158.75 0)
       (effects (font (size 1.27 1.27)) hide)
     )
@@
       (effects (font (size 1.27 1.27)) hide)
     )
-    (property "Datasheet" "" (at 40.64 116.84 0)
+    (property "Datasheet" "~" (at 40.64 116.84 0)
       (effects (font (size 1.27 1.27)) hide)
     )
@@
       (effects (font (size 1.27 1.27)) hide)
     )
-    (property "Datasheet" "" (at 63.5 120.65 0)
+    (property "Datasheet" "~" (at 63.5 120.65 0)
       (effects (font (size 1.27 1.27)) hide)
     )
@@
       (effects (font (size 1.27 1.27)) hide)
     )
-    (property "Datasheet" "" (at 68.58 120.65 0)
+    (property "Datasheet" "~" (at 68.58 120.65 0)
       (effects (font (size 1.27 1.27)) hide)
     )
@@
       (effects (font (size 1.27 1.27)) hide)
     )
-    (property "Datasheet" "" (at 151.13 137.16 0)
+    (property "Datasheet" "~" (at 151.13 137.16 0)
       (effects (font (size 1.27 1.27)) hide)
     )
@@
       (effects (font (size 1.27 1.27)) hide)
     )
-    (property "Datasheet" "" (at 146.05 137.16 0)
+    (property "Datasheet" "~" (at 146.05 137.16 0)
       (effects (font (size 1.27 1.27)) hide)
     )
@@
       (effects (font (size 1.524 1.524)) (justify right))
     )
-    (pin "END_MAXCOUNT" output (at 260.35 90.17 0)
-      (effects (font (size 1.524 1.524)) (justify right))
-    )
-    (pin "NEXT_AFTERSET" output (at 260.35 87.63 0)
-      (effects (font (size 1.524 1.524)) (justify right))
-    )
-    (pin "END_ISIMPLE" output (at 260.35 92.71 0)
-      (effects (font (size 1.524 1.524)) (justify right))
-    )
     (pin "OPCHOOSE_CLK" output (at 260.35 63.5 0)
       (effects (font (size 1.524 1.524)) (justify right))
     )
     (pin "BCFG_SPI_CLK" output (at 260.35 130.81 0)
-      (effects (font (size 1.524 1.524)) (justify right))
-    )
-    (pin "NEXT_ISIMPLE" output (at 260.35 95.25 0)
       (effects (font (size 1.524 1.524)) (justify right))
     )
@@
       (effects (font (size 1.524 1.524)) (justify right))
     )
+    (pin "REQ_END_MAXSEQ" output (at 260.35 90.17 0)
+      (effects (font (size 1.524 1.524)) (justify right))
+    )
+    (pin "REQ_NEXT_AFTERISET" output (at 260.35 87.63 0)
+      (effects (font (size 1.524 1.524)) (justify right))
+    )
+    (pin "REQ_NEXT_ISIMPLE" output (at 260.35 95.25 0)
+      (effects (font (size 1.524 1.524)) (justify right))
+    )
+    (pin "REQ_END_ISIMPLE" output (at 260.35 92.71 0)
+      (effects (font (size 1.524 1.524)) (justify right))
+    )

Commit message: replacing 10k pull-ups resistors with 1k in order to limit the effect on rise up time
Parts:
- R1, R2, R3, R6, R7: value 10k -> 1k
Changed lines of the file:
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@@
       (effects (font (size 1.27 1.27)))
     )
-    (property "Value" "10k" (at 140.97 137.16 90)
+    (property "Value" "1k" (at 140.97 137.16 90)
       (effects (font (size 1.27 1.27)))
     )
@@
       (effects (font (size 1.27 1.27)))
     )
-    (property "Value" "10k" (at 63.5 120.65 90)
+    (property "Value" "1k" (at 63.5 120.65 90)
       (effects (font (size 1.27 1.27)))
     )
@@
       (effects (font (size 1.27 1.27)))
     )
-    (property "Value" "10k" (at 68.58 120.65 90)
+    (property "Value" "1k" (at 68.58 120.65 90)
       (effects (font (size 1.27 1.27)))
     )
@@
       (effects (font (size 1.27 1.27)))
     )
-    (property "Value" "10k" (at 151.13 137.16 90)
+    (property "Value" "1k" (at 151.13 137.16 90)
       (effects (font (size 1.27 1.27)))
     )
@@
       (effects (font (size 1.27 1.27)))
     )
-    (property "Value" "10k" (at 146.05 137.16 90)
-      (effects (font (size 1.27 1.27)))
-    )
+    (property "Value" "1k" (at 146.05 137.16 90)
+      (effects (font (size 1.27 1.27)))
+    )
