File: fileRAM.kicad_sch (KiCad schematic)
At the start: 13 parts, among them J3 MM1_5530843-2, U34 74LVC1G34, U35 74AHC273, U36 74AHC1G04, U37 74AHC273, U38 74AHC374, U39 74AHC1G04

Commit message: update BOM
Parts:
- U35, U37: footprint Package_SO:SOIC-20W_7.5x12.8mm_P1.27mm -> Package_SO:SSOP-20_5.3x7.2mm_P0.65mm
Changed lines of the file:
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@@
       (effects (font (size 1.27 1.27)))
     )
-    (property "Footprint" "Package_SO:SOIC-20W_7.5x12.8mm_P1.27mm" (at 50.8 138.43 0)
+    (property "Footprint" "Package_SO:SSOP-20_5.3x7.2mm_P0.65mm" (at 50.8 138.43 0)
       (effects (font (size 1.27 1.27)) hide)
     )
@@
       (effects (font (size 1.27 1.27)))
     )
-    (property "Footprint" "Package_SO:SOIC-20W_7.5x12.8mm_P1.27mm" (at 119.38 138.43 0)
+    (property "Footprint" "Package_SO:SSOP-20_5.3x7.2mm_P0.65mm" (at 119.38 138.43 0)
       (effects (font (size 1.27 1.27)) hide)
     )
